File: PCB/Sub-Board/slots.kicad_sch (KiCad schematic)
At the start: 136 parts, among them J10 Type, J11 Power/I2C, J12 Address, J13 Power/I2C, J14 Address, J15 GPIO, J16 Type, J17 GPIO, J18 Type, J19 Power/I2C, J20 Address, J21 Power/I2C, J22 Address, J23 GPIO, J24 Type, J25 GPIO, J26 Type, J27 Power/I2C, J28 Address, J29 Power/I2C, J3 Power/I2C, J30 Address, J31 GPIO, J32 Type, J33 GPIO, J34 Type, J4 Address, J5 Power/I2C, J6 Address, J7 GPIO, J8 Type, J9 GPIO

Commit message: Sub Board PCB: Pin Connectors
Parts:
- J10, J12, J14, J16, J18, J20, J22, J24, J26, J28, J30, J32, J34, J4, J6, J8: footprint Connector_PinHeader_1.27mm:PinHeader_1x04_P1.27mm_Vertical -> Connector_PinSocket_1.27mm:PinSocket_1x04_P1.27mm_Vertical
- J11, J13, J19, J21, J27, J29, J3, J5: footprint Connector_PinHeader_1.27mm:PinHeader_1x05_P1.27mm_Vertical -> Connector_PinSocket_1.27mm:PinSocket_1x05_P1.27mm_Vertical
- J15, J17, J23, J25, J31, J33, J7, J9: footprint Connector_PinHeader_1.27mm:PinHeader_1x06_P1.27mm_Vertical -> Connector_PinSocket_1.27mm:PinSocket_1x06_P1.27mm_Vertical
Changed lines of the file:
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@@
 			)
 		)
-		(property "Footprint" "Connector_PinHeader_1.27mm:PinHeader_1x04_P1.27mm_Vertical"
+		(property "Footprint" "Connector_PinSocket_1.27mm:PinSocket_1x04_P1.27mm_Vertical"
 			(at 248.92 114.3 0)
 			(effects
@@
 			)
 		)
-		(property "Footprint" "Connector_PinHeader_1.27mm:PinHeader_1x05_P1.27mm_Vertical"
+		(property "Footprint" "Connector_PinSocket_1.27mm:PinSocket_1x05_P1.27mm_Vertical"
 			(at 81.28 168.91 0)
 			(effects
@@
 			)
 		)
-		(property "Footprint" "Connector_PinHeader_1.27mm:PinHeader_1x06_P1.27mm_Vertical"
+		(property "Footprint" "Connector_PinSocket_1.27mm:PinSocket_1x06_P1.27mm_Vertical"
 			(at 327.66 72.39 0)
 			(effects
@@
 			)
 		)
-		(property "Footprint" "Connector_PinHeader_1.27mm:PinHeader_1x05_P1.27mm_Vertical"
+		(property "Footprint" "Connector_PinSocket_1.27mm:PinSocket_1x05_P1.27mm_Vertical"
 			(at 241.3 72.39 0)
 			(effects
@@
 			)
 		)
-		(property "Footprint" "Connector_PinHeader_1.27mm:PinHeader_1x06_P1.27mm_Vertical"
+		(property "Footprint" "Connector_PinSocket_1.27mm:PinSocket_1x06_P1.27mm_Vertical"
 			(at 248.92 168.91 0)
 			(effects
@@
 			)
 		)
-		(property "Footprint" "Connector_PinHeader_1.27mm:PinHeader_1x04_P1.27mm_Vertical"
+		(property "Footprint" "Connector_PinSocket_1.27mm:PinSocket_1x04_P1.27mm_Vertical"
 			(at 88.9 114.3 0)
 			(effects
@@
 			)
 		)
-		(property "Footprint" "Connector_PinHeader_1.27mm:PinHeader_1x06_P1.27mm_Vertical"
+		(property "Footprint" "Connector_PinSocket_1.27mm:PinSocket_1x06_P1.27mm_Vertical"
 			(at 88.9 168.91 0)
 			(effects
@@
 			)
 		)
-		(property "Footprint" "Connector_PinHeader_1.27mm:PinHeader_1x06_P1.27mm_Vertical"
+		(property "Footprint" "Connector_PinSocket_1.27mm:PinSocket_1x06_P1.27mm_Vertical"
 			(at 327.66 168.91 0)
 			(effects
@@
 			)
 		)
-		(property "Footprint" "Connector_PinHeader_1.27mm:PinHeader_1x04_P1.27mm_Vertical"
+		(property "Footprint" "Connector_PinSocket_1.27mm:PinSocket_1x04_P1.27mm_Vertical"
 			(at 327.66 114.3 0)
 			(effects
@@
 			)
 		)
-		(property "Footprint" "Connector_PinHeader_1.27mm:PinHeader_1x04_P1.27mm_Vertical"
+		(property "Footprint" "Connector_PinSocket_1.27mm:PinSocket_1x04_P1.27mm_Vertical"
 			(at 241.3 114.3 0)
 			(effects
@@
 			)
 		)
-		(property "Footprint" "Connector_PinHeader_1.27mm:PinHeader_1x06_P1.27mm_Vertical"
+		(property "Footprint" "Connector_PinSocket_1.27mm:PinSocket_1x06_P1.27mm_Vertical"
 			(at 88.9 72.39 0)
 			(effects
@@
 			)
 		)
-		(property "Footprint" "Connector_PinHeader_1.27mm:PinHeader_1x05_P1.27mm_Vertical"
+		(property "Footprint" "Connector_PinSocket_1.27mm:PinSocket_1x05_P1.27mm_Vertical"
 			(at 161.29 72.39 0)
 			(effects
@@
 			)
 		)
-		(property "Footprint" "Connector_PinHeader_1.27mm:PinHeader_1x04_P1.27mm_Vertical"
+		(property "Footprint" "Connector_PinSocket_1.27mm:PinSocket_1x04_P1.27mm_Vertical"
 			(at 161.29 210.82 0)
 			(effects
@@
 			)
 		)
-		(property "Footprint" "Connector_PinHeader_1.27mm:PinHeader_1x04_P1.27mm_Vertical"
+		(property "Footprint" "Connector_PinSocket_1.27mm:PinSocket_1x04_P1.27mm_Vertical"
 			(at 320.04 210.82 0)
 			(effects
@@
 			)
 		)
-		(property "Footprint" "Connector_PinHeader_1.27mm:PinHeader_1x05_P1.27mm_Vertical"
+		(property "Footprint" "Connector_PinSocket_1.27mm:PinSocket_1x05_P1.27mm_Vertical"
 			(at 241.3 168.91 0)
 			(effects
@@
 			)
 		)
-		(property "Footprint" "Connector_PinHeader_1.27mm:PinHeader_1x04_P1.27mm_Vertical"
+		(property "Footprint" "Connector_PinSocket_1.27mm:PinSocket_1x04_P1.27mm_Vertical"
 			(at 168.91 210.82 0)
 			(effects
@@
 			)
 		)
-		(property "Footprint" "Connector_PinHeader_1.27mm:PinHeader_1x04_P1.27mm_Vertical"
+		(property "Footprint" "Connector_PinSocket_1.27mm:PinSocket_1x04_P1.27mm_Vertical"
 			(at 168.91 114.3 0)
 			(effects
@@
 			)
 		)
-		(property "Footprint" "Connector_PinHeader_1.27mm:PinHeader_1x05_P1.27mm_Vertical"
+		(property "Footprint" "Connector_PinSocket_1.27mm:PinSocket_1x05_P1.27mm_Vertical"
 			(at 81.28 72.39 0)
 			(effects
@@
 			)
 		)
-		(property "Footprint" "Connector_PinHeader_1.27mm:PinHeader_1x04_P1.27mm_Vertical"
+		(property "Footprint" "Connector_PinSocket_1.27mm:PinSocket_1x04_P1.27mm_Vertical"
 			(at 88.9 210.82 0)
 			(effects
@@
 			)
 		)
-		(property "Footprint" "Connector_PinHeader_1.27mm:PinHeader_1x06_P1.27mm_Vertical"
+		(property "Footprint" "Connector_PinSocket_1.27mm:PinSocket_1x06_P1.27mm_Vertical"
 			(at 168.91 168.91 0)
 			(effects
@@
 			)
 		)
-		(property "Footprint" "Connector_PinHeader_1.27mm:PinHeader_1x06_P1.27mm_Vertical"
+		(property "Footprint" "Connector_PinSocket_1.27mm:PinSocket_1x06_P1.27mm_Vertical"
 			(at 248.92 72.39 0)
 			(effects
@@
 			)
 		)
-		(property "Footprint" "Connector_PinHeader_1.27mm:PinHeader_1x05_P1.27mm_Vertical"
+		(property "Footprint" "Connector_PinSocket_1.27mm:PinSocket_1x05_P1.27mm_Vertical"
 			(at 320.04 168.91 0)
 			(effects
@@
 			)
 		)
-		(property "Footprint" "Connector_PinHeader_1.27mm:PinHeader_1x04_P1.27mm_Vertical"
+		(property "Footprint" "Connector_PinSocket_1.27mm:PinSocket_1x04_P1.27mm_Vertical"
 			(at 248.92 210.82 0)
 			(effects
@@
 			)
 		)
-		(property "Footprint" "Connector_PinHeader_1.27mm:PinHeader_1x04_P1.27mm_Vertical"
+		(property "Footprint" "Connector_PinSocket_1.27mm:PinSocket_1x04_P1.27mm_Vertical"
 			(at 241.3 210.82 0)
 			(effects
@@
 			)
 		)
-		(property "Footprint" "Connector_PinHeader_1.27mm:PinHeader_1x04_P1.27mm_Vertical"
+		(property "Footprint" "Connector_PinSocket_1.27mm:PinSocket_1x04_P1.27mm_Vertical"
 			(at 320.04 114.3 0)
 			(effects
@@
 			)
 		)
-		(property "Footprint" "Connector_PinHeader_1.27mm:PinHeader_1x04_P1.27mm_Vertical"
+		(property "Footprint" "Connector_PinSocket_1.27mm:PinSocket_1x04_P1.27mm_Vertical"
 			(at 161.29 114.3 0)
 			(effects
@@
 			)
 		)
-		(property "Footprint" "Connector_PinHeader_1.27mm:PinHeader_1x05_P1.27mm_Vertical"
+		(property "Footprint" "Connector_PinSocket_1.27mm:PinSocket_1x05_P1.27mm_Vertical"
 			(at 320.04 72.39 0)
 			(effects
@@
 			)
 		)
-		(property "Footprint" "Connector_PinHeader_1.27mm:PinHeader_1x04_P1.27mm_Vertical"
+		(property "Footprint" "Connector_PinSocket_1.27mm:PinSocket_1x04_P1.27mm_Vertical"
 			(at 327.66 210.82 0)
 			(effects
@@
 			)
 		)
-		(property "Footprint" "Connector_PinHeader_1.27mm:PinHeader_1x04_P1.27mm_Vertical"
+		(property "Footprint" "Connector_PinSocket_1.27mm:PinSocket_1x04_P1.27mm_Vertical"
 			(at 81.28 210.82 0)
 			(effects
@@
 			)
 		)
-		(property "Footprint" "Connector_PinHeader_1.27mm:PinHeader_1x05_P1.27mm_Vertical"
+		(property "Footprint" "Connector_PinSocket_1.27mm:PinSocket_1x05_P1.27mm_Vertical"
 			(at 161.29 168.91 0)
 			(effects
@@
 			)
 		)
-		(property "Footprint" "Connector_PinHeader_1.27mm:PinHeader_1x04_P1.27mm_Vertical"
+		(property "Footprint" "Connector_PinSocket_1.27mm:PinSocket_1x04_P1.27mm_Vertical"
 			(at 81.28 114.3 0)
 			(effects
@@
 			)
 		)
-		(property "Footprint" "Connector_PinHeader_1.27mm:PinHeader_1x06_P1.27mm_Vertical"
+		(property "Footprint" "Connector_PinSocket_1.27mm:PinSocket_1x06_P1.27mm_Vertical"
 			(at 168.91 72.39 0)
 			(effects

Commit message: Sub Board PCB: GND/GNDD
Connections:
- net GND: no longer R100.1, R101.1, R102.1, R103.1, R109.2, R110.2, R111.2, R112.1, R113.1, R114.1, R115.1, R116.1, R117.1, R118.1, R119.1, R120.1, R121.1, R122.1, R123.1, R124.1, R125.1, R126.1, R127.1, R128.1, R129.1, R27.2, R28.2, R29.2, R30.2, R31.2, R32.2, R33.2, R34.1, R35.1, R36.1, R37.1, R38.1, R39.1, R40.1, R41.1, R42.1, R43.1, R44.1, R45.1, R46.1, R47.1, R48.1, R49.1, R50.1, R51.1, R55.2, R56.2, R57.2, R58.2, R59.2, R60.1, R61.1, R62.1, R63.1, R64.1, R65.1, R66.1, R67.1, R68.1, R69.1, R70.1, R71.1, R72.1, R73.1, R74.1, R75.1, R76.1, R77.1, R81.2, R82.2, R83.2, R84.2, R85.2, R86.1, R87.1, R88.1, R89.1, R90.1, R91.1, R92.1, R93.1, R94.1, R95.1, R96.1, R97.1, R98.1, R99.1
- new net GNDD: R100.1, R101.1, R102.1, R103.1, R109.2, R110.2, R111.2, R112.1, R113.1, R114.1, R115.1, R116.1, R117.1, R118.1, R119.1, R120.1, R121.1, R122.1, R123.1, R124.1, R125.1, R126.1, R127.1, R128.1, R129.1, R27.2, R28.2, R29.2, R30.2, R31.2, R32.2, R33.2, R34.1, R35.1, R36.1, R37.1, R38.1, R39.1, R40.1, R41.1, R42.1, R43.1, R44.1, R45.1, R46.1, R47.1, R48.1, R49.1, R50.1, R51.1, R55.2, R56.2, R57.2, R58.2, R59.2, R60.1, R61.1, R62.1, R63.1, R64.1, R65.1, R66.1, R67.1, R68.1, R69.1, R70.1, R71.1, R72.1, R73.1, R74.1, R75.1, R76.1, R77.1, R81.2, R82.2, R83.2, R84.2, R85.2, R86.1, R87.1, R88.1, R89.1, R90.1, R91.1, R92.1, R93.1, R94.1, R95.1, R96.1, R97.1, R98.1, R99.1

Commit message: Sub Board PCB: Routing (wip)
Connections:
- net GNDD is gone; now on net GND: R100.1, R101.1, R102.1, R103.1, R109.2, R110.2, R111.2, R112.1, R113.1, R114.1, R115.1, R116.1, R117.1, R118.1, R119.1, R120.1, R121.1, R122.1, R123.1, R124.1, R125.1, R126.1, R127.1, R128.1, R129.1, R27.2, R28.2, R29.2, R30.2, R31.2, R32.2, R33.2, R34.1, R35.1, R36.1, R37.1, R38.1, R39.1, R40.1, R41.1, R42.1, R43.1, R44.1, R45.1, R46.1, R47.1, R48.1, R49.1, R50.1, R51.1, R55.2, R56.2, R57.2, R58.2, R59.2, R60.1, R61.1, R62.1, R63.1, R64.1, R65.1, R66.1, R67.1, R68.1, R69.1, R70.1, R71.1, R72.1, R73.1, R74.1, R75.1, R76.1, R77.1, R81.2, R82.2, R83.2, R84.2, R85.2, R86.1, R87.1, R88.1, R89.1, R90.1, R91.1, R92.1, R93.1, R94.1, R95.1, R96.1, R97.1, R98.1, R99.1
Changed lines of the file:
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@@
 			)
 		)
-		(property "Value" "GNDD"
+		(property "Value" "GND"
 			(at 81.28 234.0031 0)
 			(effects
@@
 			)
 		)
-		(property "Value" "GNDD"
+		(property "Value" "GND"
 			(at 168.91 234.0031 0)
 			(effects
@@
 			)
 		)
-		(property "Value" "GNDD"
+		(property "Value" "GND"
 			(at 320.04 234.0031 0)
 			(effects
@@
 			)
 		)
-		(property "Value" "GNDD"
+		(property "Value" "GND"
 			(at 327.66 234.0031 0)
 			(effects
@@
 			)
 		)
-		(property "Value" "GNDD"
+		(property "Value" "GND"
 			(at 168.91 197.1731 0)
 			(effects
@@
 			)
 		)
-		(property "Value" "GNDD"
+		(property "Value" "GND"
 			(at 241.3 234.0031 0)
 			(effects
@@
 			)
 		)
-		(property "Value" "GNDD"
+		(property "Value" "GND"
 			(at 327.66 197.1731 0)
 			(effects
@@
 			)
 		)
-		(property "Value" "GNDD"
+		(property "Value" "GND"
 			(at 327.66 137.4831 0)
 			(effects
@@
 			)
 		)
-		(property "Value" "GNDD"
+		(property "Value" "GND"
 			(at 88.9 137.4831 0)
 			(effects
@@
 			)
 		)
-		(property "Value" "GNDD"
+		(property "Value" "GND"
 			(at 88.9 234.0031 0)
 			(effects
@@
 			)
 		)
-		(property "Value" "GNDD"
+		(property "Value" "GND"
 			(at 248.92 234.0031 0)
 			(effects
@@
 			)
 		)
-		(property "Value" "GNDD"
+		(property "Value" "GND"
 			(at 241.3 137.4831 0)
 			(effects
@@
 			)
 		)
-		(property "Value" "GNDD"
+		(property "Value" "GND"
 			(at 248.92 197.1731 0)
 			(effects
@@
 			)
 		)
-		(property "Value" "GNDD"
+		(property "Value" "GND"
 			(at 161.29 137.4831 0)
 			(effects
@@
 			)
 		)
-		(property "Value" "GNDD"
+		(property "Value" "GND"
 			(at 327.66 100.6531 0)
 			(effects
@@
 			)
 		)
-		(property "Value" "GNDD"
+		(property "Value" "GND"
 			(at 168.91 137.4831 0)
 			(effects
@@
 			)
 		)
-		(property "Value" "GNDD"
+		(property "Value" "GND"
 			(at 320.04 137.4831 0)
 			(effects
@@
 			)
 		)
-		(property "Value" "GNDD"
+		(property "Value" "GND"
 			(at 88.9 197.1731 0)
 			(effects
@@
 			)
 		)
-		(property "Value" "GNDD"
+		(property "Value" "GND"
 			(at 248.92 100.6531 0)
 			(effects
@@
 			)
 		)
-		(property "Value" "GNDD"
+		(property "Value" "GND"
 			(at 248.92 137.4831 0)
 			(effects
@@
 			)
 		)
-		(property "Value" "GNDD"
+		(property "Value" "GND"
 			(at 81.28 137.4831 0)
 			(effects
@@
 			)
 		)
-		(property "Value" "GNDD"
+		(property "Value" "GND"
 			(at 88.9 100.6531 0)
 			(effects
@@
 			)
 		)
-		(property "Value" "GNDD"
+		(property "Value" "GND"
 			(at 168.91 100.6531 0)
 			(effects
@@
 			)
 		)
-		(property "Value" "GNDD"
+		(property "Value" "GND"
 			(at 161.29 234.0031 0)
 			(effects
