File: PCB/Sub-Board/KiCAD/address_selector.kicad_sch (KiCad schematic)
At the start: 10 parts, among them SW1 SW_DIP_x07

Commit message: PCB Sub Board: Revision 2
Parts:
- SW1: value SW_DIP_x07 -> CTS 219-7LPSTR
Changed lines of the file:
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@@
 	(title_block
 		(title "Modular Music Controller / Sub-Board / Address Selector")
-		(date "2025-11-02")
-		(rev "1")
+		(date "2025-12-02")
+		(rev "2")
 		(company "Dennis Schulmeister-Zimolong")
 	)
@@
 		(fields_autoplaced yes)
 		(property "Reference" "SW1"
-			(at 55.88 55.5455 0)
-			(effects
-				(font
-					(size 1.27 1.27)
-				)
-			)
-		)
-		(property "Value" "SW_DIP_x07"
+			(at 55.88 57.9699 0)
+			(effects
+				(font
+					(size 1.27 1.27)
+				)
+			)
+		)
+		(property "Value" "CTS 219-7LPSTR"
 			(at 55.88 57.9698 0)
 			(effects
@@
 					(size 1.27 1.27)
 				)
-			)
-		)
+				(hide yes)
+			)
+		)
