File: PCB/Sub-Board/KiCAD/power_supply.kicad_sch (KiCad schematic)
At the start: 7 parts, among them U1 TPS629210DRLR

Commit message: PCB Sub Board: Revision 2
Parts:
- FB1: value 600Ω @ 100MHz ~300-500mA -> Laird HZ0603C651R-10
Other:
- note added: "650Ω @ 100MHz ~300mA"
Changed lines of the file:
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@@
 	(title_block
 		(title "Modular Music Controller / Sub-Board / Power Supply")
-		(date "2025-11-02")
-		(rev "1")
+		(date "2025-12-02")
+		(rev "2")
 		(company "Dennis Schulmeister-Zimolong")
+	)
+	(text "650Ω @ 100MHz ~300mA"
+		(exclude_from_sim no)
+		(at 182.88 66.04 0)
+		(effects
+			(font
+				(size 1.27 1.27)
+			)
+		)
 	)
 	(text "Power Supply"
@@
 			)
 		)
-		(property "Value" "600Ω @ 100MHz ~300-500mA"
+		(property "Value" "Laird HZ0603C651R-10"
 			(at 181.5592 65.4882 90)
 			(effects
@@
 					(size 1.27 1.27)
 				)
+				(hide yes)
 			)
 		)
@@
 			)
 		)
-		(property "Description" "Ferrite bead"
+		(property "Description" "Ferrite bead - 650Ω @ 100MHz ~300-500mA"
 			(at 181.61 69.85 0)
 			(effects
