File: PCB/Sub-Board/KiCAD/slots.kicad_sch (KiCad schematic)
At the start: 136 parts, among them J10 Type, J11 Power/I2C, J12 Address, J13 Power/I2C, J14 Address, J15 GPIO, J16 Type, J17 GPIO, J18 Type, J19 Power/I2C, J20 Address, J21 Power/I2C, J22 Address, J23 GPIO, J24 Type, J25 GPIO, J26 Type, J27 Power/I2C, J28 Address, J29 Power/I2C, J3 Power/I2C, J30 Address, J31 GPIO, J32 Type, J33 GPIO, J34 Type, J4 Address, J5 Power/I2C, J6 Address, J7 GPIO, J8 Type, J9 GPIO

Commit message: PCB Sub Board: Revision 2
Parts:
- J10, J16, J18, J24, J26, J32, J34, J8: value Type -> Samtec RSM-104-02-L-S
- J11, J13, J19, J21, J27, J29, J3, J5: value Power/I2C -> Samtec RSM-105-02-L-S
- J12, J14, J20, J22, J28, J30, J4, J6: value Address -> Samtec RSM-104-02-L-S
- J15, J17, J23, J25, J31, J33, J7, J9: value GPIO -> Samtec RSM-106-02-L-S
Other:
- note added: "Address"
- note added: "GPIO"
- note added: "Power/I2C"
- note added: "Type"
