File: PCB/Sub-Board/KiCAD/stm32-mcu.kicad_sch (KiCad schematic)
At the start: 42 parts, among them J2 Conn_01x04_Pin, U2 74HC165, U3 STM32F401VETx, U4 74HC165, U5 74HC165, U6 74HC165, U7 74HC165, Y1 26 MHz

Commit message: PCB Sub Board: Revision 2
Parts:
- removed Y1: 26 MHz, Crystal:Crystal_SMD_3215-2Pin_3.2x1.5mm, symbol Device:Crystal
- added Y1: Kyocera CX2016DB26000H0FLJC2, CX2016DB26000H0FLJC2:OSC_CX2016DB26000H0FLJC2, symbol CX2016DB26000H0FLJC2:CX2016DB26000H0FLJC2
- J2: value Conn_01x04_Pin -> Harwin M20-8770446
- U2, U4, U5, U6, U7: value 74HC165 -> Nexperia 74HC165PW,118
- U3: value STM32F401VETx -> STM32F401VET6
Connections:
- net GND: now also Y1.2 (GND)
- net PH0: now also Y1.1
- net PH1: now also Y1.3
Other:
- note added: "26 MHz"
- note added: "74HC165"
- moved on the sheet: C14, C21, C24, J2, R20, R21, R23, R24
