File: PCB/Sub-Board/KiCAD/system_bus.kicad_sch (KiCad schematic)
At the start: 5 parts, among them J1 Conn_02x08

Commit message: PCB Sub Board: Revision 2
Parts:
- J1: value Conn_02x08 -> Harwin M20-8760846
- L1: value Choke_Wurth_WE-CNSW_744232090 -> Wuerth 744232090
Changed lines of the file:
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@@
 	(title_block
 		(title "Modular Music Controller / Sub-Board / System Bus")
-		(date "2025-11-02")
-		(rev "1")
+		(date "2025-12-02")
+		(rev "2")
 		(company "Dennis Schulmeister-Zimolong")
 	)
@@
 		(fields_autoplaced yes)
 		(property "Reference" "J1"
-			(at 80.01 59.3555 0)
-			(effects
-				(font
-					(size 1.27 1.27)
-				)
-			)
-		)
-		(property "Value" "Conn_02x08"
+			(at 80.01 61.7799 0)
+			(effects
+				(font
+					(size 1.27 1.27)
+				)
+			)
+		)
+		(property "Value" "Harwin M20-8760846"
 			(at 80.01 61.7798 0)
 			(effects
@@
 					(size 1.27 1.27)
 				)
+				(hide yes)
 			)
 		)
@@
 			)
 		)
-		(property "Description" "TPD2E001 SOP23 package"
+		(property "Description" "TPD2E001 SOP23 package (alternatively TPD2E2U06DRLR)"
 			(at 149.86 106.68 0)
 			(effects
@@
 			)
 		)
-		(property "Value" "Choke_Wurth_WE-CNSW_744232090"
+		(property "Value" "Wuerth 744232090"
 			(at 184.15 58.674 0)
 			(effects
@@
 					(size 1.27 1.27)
 				)
-			)
-		)
+				(hide yes)
+			)
+		)
