File: PCB/Block-Simple-Switch/KiCAD/Block-Simple-Switch.kicad_pcb (KiCad board)
At the start: 2 copper layers, 24.1 x 24.1 mm, 12 parts, among them J1 Samtec MTMS-105-02-T-S-100, J2 Samtec MTMS-104-02-T-S-100, J3 Samtec MTMS-106-02-T-S-100, J3 Samtec RSM-105-02-L-S, J4 Samtec MTMS-104-02-T-S-100, J4 Samtec RSM-104-02-L-S, J7 Samtec RSM-106-02-L-S, J8 Samtec RSM-104-02-L-S, SW1 SW_Push

Commit message: PCB Block Simple Switch (finished)
Parts:
- removed the J3 at (128.5, 103.1)
- removed the J4 at (149.6, 124.2)
- removed J7: Samtec RSM-106-02-L-S, Connector_PinSocket_1.27mm:PinSocket_1x06_P1.27mm_Vertical
- removed J8: Samtec RSM-104-02-L-S, Connector_PinSocket_1.27mm:PinSocket_1x04_P1.27mm_Vertical
- D1: footprint LED_SMD:LED_0402_1005Metric -> LED_SMD:LED_0805_2012Metric
- J1, J2, J3, J4, R1: moved to B.Cu
- moved J4 28.9 mm to (128.5, 124.2), turned to -90 degrees
- moved J2 22.0 mm to (149.6, 124.2), turned to 0 degrees
- moved J3 13.3 mm to (149.6, 103.1), turned to 90 degrees
- moved J1 10.7 mm to (128.5, 103.1), turned to 180 degrees
- moved R2 0.91 mm to (140.0, 105.0), turned to -90 degrees
- moved D1 0.62 mm to (139.1, 107.3)
Connections:
- J1 pad 2: unconnected-(J1-Pin_2-Pad2) -> /AREF
- J1 pad 4: unconnected-(J1-Pin_4-Pad4) -> /SlotBus.Data
- J1 pad 5: unconnected-(J1-Pin_5-Pad5) -> /SlotBus.Clock
- J2 pad 1: unconnected-(J2-Pin_1-Pad1) -> /Addr0
- J2 pad 2: unconnected-(J2-Pin_2-Pad2) -> /Addr1
- J2 pad 3: unconnected-(J2-Pin_3-Pad3) -> /Addr2
- J2 pad 4: unconnected-(J2-Pin_4-Pad4) -> /Addr3
- J3 pad 2: unconnected-(J3-Pin_2-Pad2) -> /C
- J3 pad 3: unconnected-(J3-Pin_3-Pad3) -> /B
- J3 pad 5: unconnected-(J3-Pin_5-Pad5) -> /A1
- J3 pad 6: unconnected-(J3-Pin_6-Pad6) -> /A0
- J4 pad 1: unconnected-(J4-Pin_1-Pad1) -> /Typ0
- J4 pad 2: unconnected-(J4-Pin_2-Pad2) -> /Typ1
- J4 pad 3: unconnected-(J4-Pin_3-Pad3) -> /Typ2
- J4 pad 4: unconnected-(J4-Pin_4-Pad4) -> /Typ3
Routing:
- net /A: track 0.00 -> 21.1 mm
- net /+3.3V Digital: track 0.00 -> 10.5 mm
- net GND: track 0.00 -> 10.3 mm
- net /LED: track 0.00 -> 10.1 mm
- net Net-(R1-Pad2): track 0.00 -> 9.70 mm
- net Net-(D1-A): track 0.00 -> 1.83 mm
Other:
- board text added: "Modular Music Controller"
- board text added: "Switch & LED"
- board text removed: "TODO: Anordnung der Pin-Header -> Ausrichtung beachten! -> Werden von oben aufgesteckt!"
