File: PCB/Block-Simple-Switch/KiCAD/Block-Simple-Switch.kicad_sch (KiCad schematic)
At the start: 8 parts, among them J1 Samtec MTMS-105-02-T-S-100, J2 Samtec MTMS-104-02-T-S-100, J3 Samtec MTMS-106-02-T-S-100, J4 Samtec MTMS-104-02-T-S-100, SW1 SW_Push

Commit message: PCB Block Simple Switch (finished)
Parts:
- D1: footprint LED_SMD:LED_0402_1005Metric -> LED_SMD:LED_0805_2012Metric
Connections:
- net Typ0: now reaches J4.1 (Pin_1)
- net Typ1: now reaches J4.2 (Pin_2)
- net Typ2: now reaches J4.3 (Pin_3)
- net Typ3: now reaches J4.4 (Pin_4)
- net C: now reaches J3.2 (Pin_2)
- net B: now reaches J3.3 (Pin_3)
- net A1: now reaches J3.5 (Pin_5)
- net A0: now reaches J3.6 (Pin_6)
- net AREF: now reaches J1.2 (Pin_2)
- net SlotBus.Data: now reaches J1.4 (Pin_4)
- net SlotBus.Clock: now reaches J1.5 (Pin_5)
- net Addr0: now reaches J2.1 (Pin_1)
- net Addr1: now reaches J2.2 (Pin_2)
- net Addr2: now reaches J2.3 (Pin_3)
- net Addr3: now reaches J2.4 (Pin_4)
- no-connect marks 15 -> 14
