File: PCB/Block-Switch-1/KiCAD/Block-Switch-1.kicad_sch (KiCad schematic)
At the start: 8 parts, among them J1 Samtec MTMS-105-02-T-S-100, J2 Samtec MTMS-104-02-T-S-100, J3 Samtec MTMS-106-02-T-S-100, J4 Samtec MTMS-104-02-T-S-100, SW1 SW_Push

Commit message: PCBs for different blocks
Other:
- title: Modular Music Controller / Block / Simple Switch -> Modular Music Controller / Block / One Switch
Changed lines of the file:
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@@
 	(paper "A4")
 	(title_block
-		(title "Modular Music Controller / Block / Simple Switch")
+		(title "Modular Music Controller / Block / One Switch")
 		(date "2025-12-01")
 		(rev "1")
